Commit message: firstGazebo

File: yezibot_description/urdf/yezibot_base.urdf (robot description, URDF)
Before this commit: robot yezibot, 7 links, 6 joints
Links:
- link base_link: mass None -> 0.2; geometry collision cylinder length=0.10 radius=0.12; visual cylinder length=0.12 radius=0.10
- link caster_link: mass None -> 0.02; geometry collision sphere radius=0.016; visual sphere radius=0.016
- link imu_link: mass None -> 0.1; geometry collision box size=0.02 0.02 0.02; visual box size=0.02 0.02 0.02
- link laser_link: mass None -> 0.1; geometry collision cylinder length=0.02 radius=0.02; visual cylinder length=0.02 radius=0.02
- link left_wheel_link: mass None -> 0.2; geometry collision cylinder length=0.032 radius=0.04; visual cylinder length=0.032 radius=0.04
- link right_wheel_link: mass None -> 0.2; geometry collision cylinder length=0.032 radius=0.04; visual cylinder length=0.032 radius=0.04
Joints:
- joint base_joint: origin xyz=0.0 0.0 0.066 rpy=0.0 0.0 0.0 -> xyz=0.0 0.0 0.076 rpy=0.0 0.0 0.0
- joint caster_joint: origin xyz=0.06 0.0 -0.066 rpy=0.0 0.0 0.0 -> xyz=0.06 0.0 -0.06 rpy=0.0 0.0 0.0
- joint left_wheel_joint: origin xyz=-0.02 0.10 -0.06 rpy=1.57079 0.0 0.0 -> xyz=-0.02 0.10 -0.036 rpy=1.57079 0.0 0.0
- joint right_wheel_joint: origin xyz=-0.02 -0.10 -0.06 rpy=1.57079 0.0 0.0 -> xyz=-0.02 -0.10 -0.036 rpy=1.57079 0.0 0.0

Commit message: complete gazebo

File: yezibot_description/urdf/yezibot_base.urdf (robot description, URDF)
Before this commit: robot yezibot, 7 links, 6 joints
Links:
- added link ultrasonic_sensor_link
Joints:
- added joint ultrasonic_sensor_link: type fixed, parent base_link, child ultrasonic_sensor_link, origin xyz=0.0 0.0 0.076 rpy=0.0 0.0 0.0
- joint left_wheel_joint: axis 1.0 0.0 0.0 -> 0.0 0.0 1.0
- joint right_wheel_joint: axis 1.0 0.0 0.0 -> 0.0 0.0 1.0
